Commit message: Update project structure and package name

File: urdf/new_arm.urdf (robot description, URDF)
Before this commit: robot rover_arm, 7 links, 6 joints
Links:
- link base_link: geometry collision box size=0.16 0.16 0.17; visual mesh filename=package://ares_arm_simulation/meshes/base_link.stl scale=1 1 1
- link link1: geometry collision box size=0.1 0.05 0.155; visual mesh filename=package://ares_arm_simulation/meshes/link_1.stl scale=1 1 1
- link link2: geometry collision box size=0.1 0.04 0.45; visual mesh filename=package://ares_arm_simulation/meshes/link_2.stl scale=1 1 1
- link link3: geometry collision box size=0.12 0.04 0.32; visual mesh filename=package://ares_arm_simulation/meshes/link_3.stl scale=1 1 1
- link link4: geometry collision box size=0.1 0.06 0.08; visual mesh filename=package://ares_arm_simulation/meshes/link_4.stl scale=1 1 1
- link link5: geometry collision box size=0.2 0.06 0.12; visual mesh filename=package://ares_arm_simulation/meshes/link_5.stl scale=1 1 1

Commit message: Miscalculated inertia fixed, pid tuned.

File: urdf/new_arm.urdf (robot description, URDF)
Before this commit: robot rover_arm, 7 links, 6 joints
Links:
- link base_link: geometry collision box size=0.16 0.16 0.17; visual mesh filename=package://new_ares/meshes/base_link.stl scale=1 1 1
- link link1: geometry collision box size=0.1 0.05 0.155; visual mesh filename=package://new_ares/meshes/link_1.stl scale=1 1 1
- link link2: geometry collision box size=0.1 0.04 0.45; visual mesh filename=package://new_ares/meshes/link_2.stl scale=1 1 1
- link link3: geometry collision box size=0.12 0.04 0.32; visual mesh filename=package://new_ares/meshes/link_3.stl scale=1 1 1
- link link4: geometry collision box size=0.1 0.06 0.08; visual mesh filename=package://new_ares/meshes/link_4.stl scale=1 1 1
- link link5: geometry collision box size=0.2 0.06 0.12; visual mesh filename=package://new_ares/meshes/link_5.stl scale=1 1 1

Commit message: Minor URDF and pid update.

File: urdf/new_arm.urdf (robot description, URDF)
Before this commit: robot rover_arm, 7 links, 6 joints
Joints:
- joint joint1: limit (none) -> effort=100 velocity=100
